Commit message: improve camera resolution

File: cob_description/urdf/sensors/kinect.gazebo.xacro (robot description, xacro)
@@ -2,5 +2,5 @@
 <root xmlns:xacro="http://www.ros.org/wiki/xacro">
   <xacro:macro name="cob_kinect_gazebo_v0" params="name ros_topic
-                                                   update_rate:=20 data_skip:=0 height:=480 width:=640">
+                                                   update_rate:=20 data_skip:=0 height:=1024 width:=1280">
     <gazebo reference="${name}_link">
       <sensor type="depth" name="${name}_frame_sensor">
@@ -10,5 +10,5 @@
           <horizontal_fov>${62.0*M_PI/180.0}</horizontal_fov>
           <image>
-            <format>B8G8R8</format>
+            <format>R8G8B8</format>
             <width>${height}</width>
             <height>${width}</height>

File: cob_description/urdf/sensors/kinect.urdf.xacro (robot description, xacro)
@@ -2,5 +2,5 @@
 <root xmlns:xacro="http://www.ros.org/wiki/xacro">
   <xacro:include filename="$(find cob_description)/urdf/sensors/kinect.gazebo.xacro" />
-  <xacro:macro name="cob_kinect_v0" params="name parent *origin ros_topic update_rate:=20 data_skip:=0 height:=480 width:=640">
+  <xacro:macro name="cob_kinect_v0" params="name parent *origin ros_topic update_rate:=20 data_skip:=0 height:=1024 width:=1280">
     <joint name="${name}_joint" type="fixed">
       <xacro:insert_block name="origin" />
